File: Circuit/v4.kicad_pcb (KiCad board)
At the start: 2 copper layers, 30 x 50 mm, 54 parts, among them J2 AVR-ISP-6, Q1 AO3400A, U1 EL3H7(B)(TA)-G

Commit message: Updated Gerber after silkscreen change
Other:
- board text added: "9 July 2020"
- board text removed: "24 March 2020"
Changed lines of the file:
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@@
     (34 B.Paste user)
     (35 F.Paste user)
-    (36 B.SilkS user hide)
+    (36 B.SilkS user)
     (37 F.SilkS user)
     (38 B.Mask user hide)
@@
     (effects (font (size 1.5 1.5) (thickness 0.3)) (justify mirror))
   )
-  (gr_text "24 March 2020" (at 113.2176 51.7876) (layer B.SilkS)
+  (gr_text "9 July 2020" (at 113.2176 51.7876) (layer B.SilkS)
     (effects (font (size 1 1) (thickness 0.2)) (justify right mirror))
   )
